Commit message: Add DROK gripper MoveIt and Gazebo control

File: src/arm_only_description/urdf/arm_only_gripper_collision_check.urdf.xacro (robot description, xacro)
@@ -522,6 +522,6 @@
       xyz="-1 0 0" />
     <limit
-      lower="0.0" upper="2.10" effort="10" velocity="2.0" />
-      <dynamics damping="2" friction="0.3" />
+      lower="0.0" upper="4.2" effort="50" velocity="8.0" />
+      <dynamics damping="4.0" friction="1.0" />
   </joint>
   <link
@@ -560,9 +560,9 @@
     <child
       link="LEFT_PLATE" />
-    <axis
-      xyz="0 -1 0" />
+    <axis xyz="-0 -1 -0" />
     <mimic joint="JOINT7" multiplier="0.0166667" offset="0.0" />
     <limit
-      lower="0.0" upper="0.025" effort="20" velocity="0.05" />
+      lower="0.0" upper="0.070" effort="80" velocity="1.0" />
+    <dynamics damping="20.0" friction="8.0" />
   </joint>
   <link
@@ -605,5 +605,6 @@
     <mimic joint="JOINT7" multiplier="0.0166667" offset="0.0" />
     <limit
-      lower="0.0" upper="0.025" effort="20" velocity="0.05" />
+      lower="0.0" upper="0.070" effort="80" velocity="1.0" />
+    <dynamics damping="20.0" friction="8.0" />
   </joint>
   <link name="gripper_tcp"/>
@@ -613,4 +614,21 @@
     <child link="gripper_tcp" />
   </joint>
+  <!-- Gripper pose-check stabilization: prevent passive gripper parts from sagging before controllers are added -->
+  <gazebo reference="gripper_base">
+    <gravity>false</gravity>
+    <selfCollide>false</selfCollide>
+  </gazebo>
+  <gazebo reference="drive_gear">
+    <gravity>false</gravity>
+    <selfCollide>false</selfCollide>
+  </gazebo>
+  <gazebo reference="LEFT_PLATE">
+    <gravity>false</gravity>
+    <selfCollide>false</selfCollide>
+  </gazebo>
+  <gazebo reference="RIGHT_PLATE">
+    <gravity>false</gravity>
+    <selfCollide>false</selfCollide>
+  </gazebo>
   <!-- Collision tuning mode: keep whole robot static in Gazebo -->
   <gazebo>

File: src/arm_only_description/urdf/arm_only_gripper_moveit.urdf.xacro (robot description, xacro)
@@ -4,4 +4,5 @@
      For more information, please see http://wiki.ros.org/sw_urdf_exporter -->
 <robot name="arm_only_gripper" xmlns:xacro="http://www.ros.org/wiki/xacro">
+  <xacro:arg name="use_embedded_ros2_control" default="true"/>
   <link
     name="ARM_BASE_LINK">
@@ -165,8 +166,6 @@
     <child
       link="LINK2" />
-    <axis
-      xyz="0 1 0" />
-    <limit
-      lower="-3.141593" upper="3.141593" effort="35" velocity="1.2" />
+    <axis xyz="0 -1 0" />
+    <limit lower="-3.141593" upper="0.10472" effort="35" velocity="1.2" />
       <dynamics damping="2" friction="0.3" />
   </joint>
@@ -248,8 +247,6 @@
     <child
       link="LINK3" />
-    <axis
-      xyz="0 -1 0" />
-    <limit
-      lower="-3.141593" upper="3.141593" effort="35" velocity="1.2" />
+    <axis xyz="0 1 0" />
+    <limit lower="-3.228859" upper="-0.087266" effort="35" velocity="1.2" />
       <dynamics damping="2" friction="0.3" />
   </joint>
@@ -522,6 +519,6 @@
       xyz="-1 0 0" />
     <limit
-      lower="0.0" upper="2.10" effort="10" velocity="2.0" />
-      <dynamics damping="2" friction="0.3" />
+      lower="0.0" upper="4.2" effort="50" velocity="8.0" />
+      <dynamics damping="4.0" friction="1.0" />
   </joint>
   <link
@@ -560,9 +557,9 @@
     <child
       link="LEFT_PLATE" />
-    <axis
-      xyz="0 -1 0" />
+    <axis xyz="-0 -1 -0" />
     <mimic joint="JOINT7" multiplier="0.0166667" offset="0.0" />
     <limit
-      lower="0.0" upper="0.025" effort="20" velocity="0.05" />
+      lower="0.0" upper="0.070" effort="80" velocity="1.0" />
+    <dynamics damping="20.0" friction="8.0" />
   </joint>
   <link
@@ -605,5 +602,6 @@
     <mimic joint="JOINT7" multiplier="0.0166667" offset="0.0" />
     <limit
-      lower="0.0" upper="0.025" effort="20" velocity="0.05" />
+      lower="0.0" upper="0.070" effort="80" velocity="1.0" />
+    <dynamics damping="20.0" friction="8.0" />
   </joint>
   <link name="gripper_tcp"/>
@@ -614,4 +612,6 @@
   </joint>
   <!-- ROS2_CONTROL_STANDARD_START -->
+  <!-- EMBEDDED_ROS2_CONTROL_WRAP_START -->
+  <xacro:if value="$(arg use_embedded_ros2_control)">
   <ros2_control name="GazeboSystem" type="system">
     <hardware>
@@ -631,5 +631,5 @@
     </joint>
     <joint name="JOINT3">
-      <command_interface name="position"><param name="initial_value">0.0</param></command_interface>
+      <command_interface name="position" />
       <state_interface name="position"><param name="initial_value">-0.2955</param></state_interface>
       <state_interface name="velocity" />
@@ -673,4 +673,29 @@
     </joint>
   </ros2_control>
+  </xacro:if>
+  <!-- EMBEDDED_ROS2_CONTROL_WRAP_END -->
+  <!-- EMBEDDED_GAZEBO_ROS2_CONTROL_PLUGIN_WRAP_START -->
+  <xacro:if value="$(arg use_embedded_ros2_control)">
+  </xacro:if>
+  <!-- EMBEDDED_GAZEBO_ROS2_CONTROL_PLUGIN_WRAP_END -->
+  <!-- ROS2_CONTROL_STANDARD_END -->
+  <!-- Gripper pose-check stabilization: prevent passive gripper parts from sagging before controllers are added -->
+  <gazebo reference="gripper_base">
+    <gravity>false</gravity>
+    <selfCollide>false</selfCollide>
+  </gazebo>
+  <gazebo reference="drive_gear">
+    <gravity>false</gravity>
+    <selfCollide>false</selfCollide>
+  </gazebo>
+  <gazebo reference="LEFT_PLATE">
+    <gravity>false</gravity>
+    <selfCollide>false</selfCollide>
+  </gazebo>
+  <gazebo reference="RIGHT_PLATE">
+    <gravity>false</gravity>
+    <selfCollide>false</selfCollide>
+  </gazebo>
+<!-- Gazebo: fix the actual root/base links so the robot body does not float or stand up. -->
   <gazebo>
     <plugin filename="libgazebo_ros2_control.so" name="gazebo_ros2_control">
@@ -681,4 +706,3 @@
     </plugin>
   </gazebo>
-  <!-- ROS2_CONTROL_STANDARD_END -->
 </robot>
