Commit message: Calibrate real gripper feedback and MoveIt mimic motion

File: src/arm_only_description/urdf/arm_only_clean_moveit.urdf.xacro (robot description, xacro)
@@ -237,5 +237,5 @@
     <child link="LINK2" />
     <axis xyz="0 -1 0" />
-    <limit lower="-3.141593" upper="0.104720" effort="35" velocity="1.2" />
+    <limit lower="-0.5" upper="0.104720" effort="35" velocity="1.2" />
     <dynamics damping="2" friction="0.3" />
   </joint>

File: src/arm_only_description/urdf/arm_only_gripper_collision_check.urdf.xacro (robot description, xacro)
@@ -168,5 +168,5 @@
       xyz="0 1 0" />
     <limit
-      lower="-3.141593" upper="3.141593" effort="35" velocity="1.2" />
+      lower="-0.5" upper="3.141593" effort="35" velocity="1.2" />
       <dynamics damping="2" friction="0.3" />
   </joint>
@@ -522,5 +522,5 @@
       xyz="-1 0 0" />
     <limit
-      lower="0.0" upper="4.2" effort="50" velocity="8.0" />
+      lower="-1.70000" upper="45.00000" effort="50" velocity="10.0" />
       <dynamics damping="4.0" friction="1.0" />
   </joint>
@@ -560,8 +560,8 @@
     <child
       link="LEFT_PLATE" />
-    <axis xyz="-0 -1 -0" />
-    <mimic joint="JOINT7" multiplier="0.0166667" offset="0.0" />
-    <limit
-      lower="0.0" upper="0.070" effort="80" velocity="1.0" />
+    <axis xyz="0 -1 0" />
+    <mimic joint="JOINT7" multiplier="0.0017130621" offset="0.0029122056" />
+    <limit
+      lower="0.0" upper="0.08000000" effort="80" velocity="0.2" />
     <dynamics damping="20.0" friction="8.0" />
   </joint>
@@ -601,9 +601,8 @@
     <child
       link="RIGHT_PLATE" />
-    <axis
-      xyz="0 1 0" />
-    <mimic joint="JOINT7" multiplier="0.0166667" offset="0.0" />
-    <limit
-      lower="0.0" upper="0.070" effort="80" velocity="1.0" />
+    <axis xyz="0 1 0" />
+    <mimic joint="JOINT7" multiplier="0.0017130621" offset="0.0029122056" />
+    <limit
+      lower="0.0" upper="0.08000000" effort="80" velocity="0.2" />
     <dynamics damping="20.0" friction="8.0" />
   </joint>

File: src/arm_only_description/urdf/arm_only_gripper_moveit.urdf.xacro (robot description, xacro)
@@ -166,5 +166,5 @@
       link="LINK2" />
     <axis xyz="0 1 0" />
-    <limit lower="0.00000" upper="3.14159" effort="35" velocity="1.2" />
+    <limit lower="-0.5" upper="3.14159" effort="35" velocity="1.2" />
       <dynamics damping="2" friction="0.3" />
   </joint>
@@ -511,5 +511,5 @@
     <axis
       xyz="-1 0 0" />
-    <limit lower="-1.78024" upper="6.42281" effort="20" velocity="8.0" />
+    <limit lower="-1.70000" upper="45.00000" effort="20" velocity="10.0" />
       <dynamics damping="4.0" friction="1.0" />
   </joint>
@@ -549,8 +549,8 @@
     <child
       link="LEFT_PLATE" />
-    <axis xyz="-0 -1 -0" />
-    <mimic joint="JOINT7" multiplier="0.0166667" offset="0.0" />
+    <axis xyz="0 -1 0" />
+    <mimic joint="JOINT7" multiplier="0.0017130621" offset="0.0029122056" />
     <limit
-      lower="0.0" upper="0.070" effort="80" velocity="1.0" />
+      lower="0.0" upper="0.08000000" effort="80" velocity="0.2" />
     <dynamics damping="20.0" friction="8.0" />
   </joint>
@@ -590,9 +590,8 @@
     <child
       link="RIGHT_PLATE" />
-    <axis
-      xyz="0 1 0" />
-    <mimic joint="JOINT7" multiplier="0.0166667" offset="0.0" />
+    <axis xyz="0 1 0" />
+    <mimic joint="JOINT7" multiplier="0.0017130621" offset="0.0029122056" />
     <limit
-      lower="0.0" upper="0.070" effort="80" velocity="1.0" />
+      lower="0.0" upper="0.08000000" effort="80" velocity="0.2" />
     <dynamics damping="20.0" friction="8.0" />
   </joint>

File: src/arm_only_moveit_config/config/arm_only_gripper.ros2_control.xacro (robot description, xacro)
@@ -56,5 +56,6 @@
                 </state_interface>
                 <state_interface name="velocity"/>
-            </joint>
+              <limit lower="-1.70000" upper="45.00000" effort="10" velocity="10.0"/>
+</joint>
         </ros2_control>
     </xacro:macro>
