Commit message: stage4: calibrate real robot for side grasp

File: src/arm_only_description/urdf/arm_only_clean_moveit.urdf.xacro (robot description, xacro)
@@ -269,5 +269,5 @@
     <child link="LINK6" />
     <axis xyz="-1 0 0" />
-    <limit lower="0.523599" upper="5.759587" effort="35" velocity="1.2" />
+    <limit lower="-2.87729" upper="1.31150" effort="35" velocity="1.0" />
     <dynamics damping="2" friction="0.3" />
   </joint>

File: src/arm_only_description/urdf/arm_only_gripper_moveit.urdf.xacro (robot description, xacro)
@@ -309,5 +309,5 @@
     <axis
       xyz="1 0 0" />
-    <limit lower="-1.65806" upper="1.65806" effort="35" velocity="1.2" />
+    <limit lower="-5.89101" upper="2.64243" effort="35" velocity="1.2" />
       <dynamics damping="2" friction="0.3" />
   </joint>
@@ -378,5 +378,5 @@
       link="LINK5" />
     <axis xyz="0 -1 0" />
-    <limit lower="-1.22173" upper="1.22173" effort="35" velocity="1.2" />
+    <limit lower="-1.52175" upper="1.31947" effort="35" velocity="1.2" />
       <dynamics damping="2" friction="0.3" />
   </joint>
@@ -424,7 +424,5 @@
     </collision>
   </link>
-  <joint
-    name="JOINT6"
-    type="continuous">
+  <joint name="JOINT6" type="revolute">
     <origin
       xyz="0.08175 0 0"
@@ -436,5 +434,5 @@
     <axis
       xyz="-1 0 0" />
-    <limit effort="35" velocity="1.2" />
+    <limit lower="-2.87729" upper="1.31150" effort="35" velocity="1.0" />
       <dynamics damping="2" friction="0.3" />
   </joint>
@@ -472,7 +470,5 @@
     name="gripper_mount_joint"
     type="fixed">
-    <origin
-      xyz="0.04825 0 0"
-      rpy="-0.16782 0 0" />
+    <origin xyz="0.04825 0 0" rpy="0.79188 0 0" />
     <parent
       link="LINK6" />
@@ -617,5 +613,5 @@
     <joint name="JOINT2">
       <command_interface name="position" />
-      <state_interface name="position"><param name="initial_value">0.58173277828</param></state_interface>
+      <state_interface name="position"><param name="initial_value">0.385378389294</param></state_interface>
       <state_interface name="velocity" />
       <state_interface name="effort" />
@@ -647,5 +643,5 @@
     <joint name="JOINT7">
       <command_interface name="position" />
-      <state_interface name="position"><param name="initial_value">-1.78024</param></state_interface>
+      <state_interface name="position"><param name="initial_value">-1.70000</param></state_interface>
       <state_interface name="velocity" />
       <state_interface name="effort" />
